Commit message: renamed robot vacuum
Signed-off-by: Piotr Zyskowski <piotr.zyskowski@robotec.ai>

File: Assets/RoboVac/urdf/RobotVacuum_description/urdf/RobotVacuum.xacro (robot description, xacro)
@@ -1,7 +1,7 @@
 <?xml version="1.0" ?>
-<robot name="AstroVAC" xmlns:xacro="http://www.ros.org/wiki/xacro">
-<xacro:include filename="$(find AstroVAC_description)/urdf/materials.xacro" />
-<xacro:include filename="$(find AstroVAC_description)/urdf/AstroVAC.trans" />
-<xacro:include filename="$(find AstroVAC_description)/urdf/AstroVAC.gazebo" />
+<robot name="RobotVacuum" xmlns:xacro="http://www.ros.org/wiki/xacro">
+<xacro:include filename="$(find RobotVacuum_description)/urdf/materials.xacro" />
+<xacro:include filename="$(find RobotVacuum_description)/urdf/RobotVacuum.trans" />
+<xacro:include filename="$(find RobotVacuum_description)/urdf/RobotVacuum.gazebo" />
 <link name="base_link">
   <inertial>
@@ -13,5 +13,5 @@
     <origin rpy="0 0 0" xyz="0 0 0"/>
     <geometry>
-      <mesh filename="package://AstroVAC_description/meshes/base_link.stl" scale="0.001 0.001 0.001"/>
+      <mesh filename="package://RobotVacuum_description/meshes/base_link.stl" scale="0.001 0.001 0.001"/>
     </geometry>
     <material name="silver"/>
@@ -20,5 +20,5 @@
     <origin rpy="0 0 0" xyz="0 0 0"/>
     <geometry>
-      <mesh filename="package://AstroVAC_description/meshes/base_link.stl" scale="0.001 0.001 0.001"/>
+      <mesh filename="package://RobotVacuum_description/meshes/base_link.stl" scale="0.001 0.001 0.001"/>
     </geometry>
   </collision>

File: Assets/RoboVac/urdf/RobotVacuum_description/urdf/materials.xacro (robot description, xacro)
@@ -1,4 +1,4 @@
 <?xml version="1.0" ?>
-<robot name="AstroVAC" xmlns:xacro="http://www.ros.org/wiki/xacro" >
+<robot name="RobotVacuum" xmlns:xacro="http://www.ros.org/wiki/xacro" >
 <material name="silver">
   <color rgba="0.700 0.700 0.700 1.000"/>
